File: HW/ebaz4205/kicad/ebaz4205.kicad_sch (KiCad schematic)
At the start: 565 parts, among them J3 4PIN-2.54MM, J4 2*3PIN-4.2MM, J5 4PIN-2.54MM, J7 NC, J8 NC, T6 BT16B03, U12 W29N01HVSINA, U20 MMBT3904/1AM, U21 MMBT3904/1AM, U22 J37I, U23 NC, U24 IP101GA, U25 RJ45, U26 J37I, U27 J37I, U28 J37I, U30 ACOI, U31 XC7Z010-1CLG400I, U65 SGM706-SYS8, U66 EM6GD16EWKG-12H, U67 EL817, U68 EL817, U69 PC817, U7 NC, U70 PC817, U72 NC, X3 NC, X5 NC, X8 33.333MHZ, Y2 NC, Y3 25.000MHZ

Commit message: Provided KiCad schematic, split into sections.
Files from https://github.com/tpecar/nl2sch/ project, commit 4de37e25
Parts:
- C147, C2280, C2367, C2368, C2369, C2371, C2372, C2373, C2374, C2375, C2376, C2377, C2378, C2379, C2381, C2382: value 10NF -> C
- C1887, C1985, C1987, C2303, C2304, C2383, C2384, C2394, C293, C295, C304, C305, C319, C320, C321, C322, C323, C327, C333, C334, C367, C368, C369, C370, C373, C374, C375, C376, C379A, C382, C386A, C387, C393, C394, C400, C401, C659, C660, C661, C662, C664: value 100NF -> C
- C2250, C2291, C2293, C2296, C2297, C2298, C2299, C2307, C2308, C2310, C2313, C2314, C2317, C2318, C2320, C2322, C2323, C2326, C2327, C2329, C2332, C2333, C2334, C2335, C2339, C2340, C2342, C2346, C2347, C2353, C2354, C2356, C2359, C2360, C2361, C2363, C667, C668, C671, C672, C674: value 470NF -> C
- C2269, C2292, C2295, C2306, C2309, C2312, C2316, C2319, C2321, C2324, C2325, C2328, C2330, C2331, C2338, C2341, C2352, C2355, C2362, C2398, C666, C670, C673: value 3.9UF -> C
- C2285, C2287, C2300, C2302: value 100PF -> C
- C2288, C2294, C2305, C2315, C2336, C2337, C2345, C2351, C2357, C2358, C665, C669: value 51UF -> C
- C2343, C2344, C2349A, C2365, C2366, C663: value 33UF -> C
- C2349, C2370, C291, C292, C306, C307, C308, C309, C310, C384, C389, C391, C396, C398, C403, C625, C626, C82: value 10UF -> C
- C2350: value RES1 -> C
- C2385, C325: value 1NF -> C
- C2395, C2396, C2397, C2399, C2400, C2401, C2402, C2403, C2404, C2405, C2406, C2407, C2408, C2409, C294, C362, C363, C364, C366, C371, C372, C379, C386, C395, C402, C538, C628, C68, C69, C71, C845, C846, C856, C856A, C93, C94: value NC -> C
- C2410, C73: value 1UF -> C
- C289, C290, C383, C385, C390, C392, C397, C399: value 22UF -> C
- C377, C380: value 22PF -> C
- D21, D22, D23: value SS810 -> D_ALT
- D24: value NC -> D_ALT
- DATA1, DATA2, DATA3: value 2*10PIN-2.0MM -> Conn_02x10_Odd_Even
- EC2, EC6: value 470UF/16V -> CP
- EC5: value 100UF/16V -> CP
- FB10, FB14, FB15, FB16, L113: value 1.2UH -> L
- J3, J5: value 4PIN-2.54MM -> Conn_01x04
- J4: value 2*3PIN-4.2MM -> Conn_02x03_Odd_Even
- J7: value NC -> Conn_01x04
- J8: value NC -> Conn_02x07_Odd_Even
- L11, L36, L9: value 0.33UH -> L
- L29, L30: value NC -> L
- L31, L32, L33, L37, L7: value 4.7UH -> L
- LED1, LED4: value G -> LED_ALT
- LED6: value R+G -> LED_dual
- R117, R120, R122, R1279, R1347, R1348, R1364, R1365, R1372, R1388, R1406, R1409, R1411, R1485, R1493, R1497, R1498, R1499, R160, R161, R162, R163, R164, R165, R1949, R2340, R2389, R2391, R2434, R2435, R2438, R2439, R244, R2440, R2441, R2442, R2443, R2444, R2445, R2445B, R2446, R2447, R245, R2468, R247, R248, R2487, R2540, R2543, R2552, R2553, R2554, R2557, R2577, R2579, R2580, R2581, R2582, R2583, R2585, R2608, R2609, R2615, R2616, R2617, R2618, R2619, R2621, R2622, R2623, R2624, R2625, R2626, R2627, R2628, R2629, R2630, R2631, R2632, R2633, R2634, R2635, R2636, R2637, R2638, R2639, R2640, R2641, R2642, R2643, R2644, R277: value NC -> R_US
- R120A, R1344, R1361, R1413, R1415, R1418, R166, R1950, R1995, R2336, R2350, R2544, R2545, R2546, R2547, R2548, R2549, R2556, R2599, R2648, R2800: value 10K 1% -> R_US
- R1333: value 51K 5% -> R_US
- R1336: value 11.3K 1% -> R_US
- R1345, R1346, R1362, R1363, R1373, R1379, R1401, R1481, R2392: value 33R 1% -> R_US
- R1358, R1359, R1360, R1502, R1503, R1507, R2469, R2470, R2560, R2645, R36, R38: value 4.7K 1% -> R_US
- R1381, R1383, R1386, R1390, R1392, R1396, R1408: value 5.1K 1% -> R_US
- R1384, R1400, R1404, R1407: value 75R 1% -> R_US
- R1385, R1391, R1394, R1397, R1405, R1410, R1487, R1488, R1491, R1492, R1504, R1505, R1506, R2436, R2437, R2461, R2462, R2463, R2464, R2465, R2466, R2472, R2473, R2473A, R2474, R2476, R2477, R2478, R2479, R2480, R2481, R2482, R2483, R2484, R2485, R2486, R2487A, R2488, R2489, R2490, R2491, R2492, R2493, R2496, R2497, R2498, R2499, R2500, R2501, R2502, R2503, R2504, R2505, R2506, R2507, R2508, R2509, R2510, R2511, R37: value 22R 1% -> R_US
- R1389, R1412, R1500, R1501: value 330R 1% -> R_US
- R1393: value 6.2K 1% -> R_US
- R1414: value 6.81K 1% -> R_US
- R1417: value 15K 1% -> R_US
- R1420: value 4.02K 1% -> R_US
- R1421: value 2K 1% -> R_US
- R1482: value 3K 5% -> R_US
- R1483: value 1.2K 5% -> R_US
- R1494, R1495, R1496, R167, R246, R2512, R2602, R2603, R2604, R2605, R2641A, R2646, R2647, R2650: value 0R 1% -> R_US
- R1948, R2430, R2432, R2433: value 100K 1% -> R_US
- R2159, R2161, R2458, R2459, R2537, R2538: value 1.2K 1% -> R_US
- R2455: value 240R 1% -> R_US
- R2456, R2457, R2542: value 80.5R 1% -> R_US
- R2460, R2471: value 0R 5% -> R_US
- R2513, R2514, R2515, R2516, R2517, R2518, R2519, R2520, R2521, R2522, R2523, R2524, R2525, R2526, R2527, R2528, R2529, R2530, R2531, R2532, R2533, R2534, R2535, R2536: value 10R 1% -> R_US
- R2539, R2541, R2578, R2584, R2586, R2587, R2588, R2590, R2598: value 20K 1% -> R_US
- R2551, R3555: value 1K 1% -> R_US
- R2558, R2559: value 1M 5% -> R_US
- R45, R46, R47: value 150R 1% -> R_US
- S2: value 6*6*5MM -> FSMRACD
- S3: value NC -> FSMRACD
- T6: value BT16B03 -> HST-0041SAR
- TP1: value 3V3 -> TestPoint
- TP2: value VDD_1V5 -> TestPoint
- TP3: value 1V8 -> TestPoint
- TP4: value 1V9 -> TestPoint
- U20, U21: value MMBT3904/1AM -> Q_NPN_BEC
- U23: value NC -> U23
- U25: value RJ45 -> 8P8C_LED
- U30: value ACOI -> TPS3839DBZ
- U31: value XC7Z010-1CLG400I -> xc7z010clg400
- U65: value SGM706-SYS8 -> SGM706
- U66: value EM6GD16EWKG-12H -> MT41K128M16JT-125_AITK
- U67, U68: value EL817 -> TLP785
- U69, U70: value PC817 -> TLP785
- U7: value NC -> Micro_SD_Card_mount
- U72: value NC -> TPS51200AQDRCRQ1
- X3: value NC -> DS1307Z+
- X5: value NC -> TXC-EBAZ
- X8: value 33.333MHZ -> TXC-7C
- Y2: value NC -> RTC_XTAL
- Y3: value 25.000MHZ -> Crystal
Other:
- note added: "DDR"
- note added: "DDR Termination"
- note added: "Data Conns"
- note added: "Ethernet PHY"
- note added: "Flash"
- note added: "Opto-Isolators"
- note added: "Power"
- note added: "RTC"
- note added: "Reset Supervisor"
- note added: "SD and Ancillary"
- note added: "Switches"
- note added: "Zynq"
- note added: "Zynq IO"
- note added: "Zynq Oscs"
- note added: "Zynq Power"

Commit message: Redrawn Schematics
The previous auto-generated schematic has been redrawn to 6* A3 pages. These schematics have been DRC'd and checked against the original converted Kicad PCB files. A few PCB changes were required to ensure correct processing. (Thanks to tpecar for helping drive this through.)
Parts:
- removed C147, C1887, C1985, C1987, C2250, C2269, C2280, C2285, C2287, C2288, C2291, C2292, C2293, C2294, C2295, C2296, C2297, C2298, C2299, C2300, C2302, C2303, C2304, C2305, C2306, C2307, C2308, C2309, C2310, C2312, C2313, C2314, C2315, C2316, C2317, C2318, C2319, C2320, C2321, C2322, C2323, C2325, C2326, C2327, C2329, C2331, C2332, C2333, C2334, C2335, C2339, C2340, C2341, C2342, C2343, C2346, C2347, C2349, C2349A, C2350, C2353, C2354, C2356, C2359, C2360, C2361, C2362, C2363, C2365, C2366, C2367, C2368, C2369, C2370, C2371, C2372, C2373, C2374, C2375, C2376, C2377, C2378, C2379, C2381, C2382, C2383, C2384, C2394, C2395, C2396, C2397, C2398, C2399, C2400, C2401, C2402, C2403, C2404, C2405, C2406, C2407, C2408, C2409, C2410, C304, C305, C307, C308, C310, C319, C322, C323, C327, C333, C334, C362, C363, C364, C366, C367, C368, C369, C370, C371, C372, C373, C374, C375, C376, C377, C379, C379A, C380, C382, C386A, C538, C659, C660, C661, C662, C663, C664, C665, C666, C667, C668, C669, C670, C671, C672, C673, C674, C68, C69, C71, C73, C856A, C93, C94: C, symbol Device:C
- removed D21, D22, D23: D_ALT, symbol Device:D_ALT
- removed DATA1, DATA2, DATA3: Conn_02x10_Odd_Even, symbol Connector_Generic:Conn_02x10_Odd_Even
- removed EC5: CP, symbol Device:CP
- removed FB10, FB15, FB16, L11, L113, L29, L30, L9: L, symbol Device:L
- removed J3, J5, J7: Conn_01x04, symbol Connector_Generic:Conn_01x04
- removed J8: Conn_02x07_Odd_Even, symbol Connector_Generic:Conn_02x07_Odd_Even
- removed LED1: LED_ALT, symbol Device:LED_ALT
- removed LED6: LED_dual, symbol ebaz4205:LED_dual
- removed R117, R120, R120A, R122, R1279, R1344, R1345, R1346, R1347, R1348, R1358, R1359, R1360, R1361, R1362, R1363, R1364, R1365, R1372, R1379, R1381, R1383, R1384, R1385, R1386, R1388, R1389, R1390, R1391, R1392, R1393, R1394, R1396, R1397, R1400, R1401, R1404, R1405, R1406, R1407, R1408, R1409, R1410, R1411, R1412, R1481, R1482, R1483, R1485, R1487, R1488, R1491, R1492, R1493, R1494, R1495, R1496, R1497, R1498, R1499, R1500, R1501, R1502, R1503, R1504, R1505, R1506, R1507, R160, R161, R162, R163, R164, R165, R166, R167, R1948, R1949, R1950, R1995, R2159, R2161, R2336, R2340, R2350, R2389, R2391, R2392, R2430, R2432, R2433, R2434, R2435, R2436, R2437, R2438, R2439, R244, R2440, R2441, R2442, R2443, R2444, R2445, R2445B, R2446, R2447, R245, R2455, R2456, R2457, R2458, R2459, R246, R2460, R2461, R2462, R2463, R2464, R2465, R2466, R2469, R247, R2470, R2472, R2473, R2473A, R2474, R2476, R2477, R2478, R2479, R248, R2480, R2481, R2482, R2483, R2484, R2485, R2486, R2487A, R2488, R2489, R2490, R2491, R2492, R2493, R2496, R2497, R2498, R2499, R2500, R2501, R2502, R2503, R2504, R2505, R2506, R2507, R2508, R2509, R2510, R2511, R2512, R2513, R2514, R2515, R2516, R2517, R2518, R2519, R2520, R2521, R2522, R2523, R2524, R2525, R2526, R2527, R2528, R2529, R2530, R2531, R2532, R2533, R2534, R2535, R2536, R2537, R2538, R2539, R2540, R2541, R2542, R2543, R2544, R2545, R2546, R2547, R2548, R2549, R2551, R2552, R2553, R2554, R2556, R2557, R2560, R2577, R2578, R2579, R2580, R2581, R2582, R2583, R2584, R2585, R2586, R2587, R2588, R2590, R2598, R2602, R2608, R2609, R2615, R2616, R2617, R2618, R2619, R2621, R2622, R2623, R2624, R2625, R2626, R2627, R2628, R2629, R2630, R2631, R2632, R2633, R2634, R2635, R2636, R2637, R2638, R2639, R2640, R2641, R2641A, R2642, R2643, R2644, R2645, R2646, R2647, R2648, R2650, R277, R3555, R36, R37, R38, R45, R46: R_US, symbol Device:R_US
- removed S2, S3: FSMRACD, TE_Connectivity-FSMRACD-*, symbol eec:FSMRACD
- removed T6: HST-0041SAR, symbol ebaz4205:HST-0041SAR
- removed U12: W29N01HVSINA, SOP50P2000X120-48N, symbol ebaz4205:W29N01HVSINA
- removed U24: IP101GA, symbol ebaz4205:IP101GA
- removed U25: 8P8C_LED, symbol ebaz4205:8P8C_LED
- removed U30: TPS3839DBZ, Package_TO_SOT_SMD:SOT-23, symbol ebaz4205:TPS3839DBZ
- removed U31: xc7z010clg400, symbol ebaz4205:xc7z010clg400
- removed U65: SGM706, symbol ebaz4205:SGM706
- removed U66: MT41K128M16JT-125_AITK, Micron-JT-0-0-*, symbol ebaz4205:MT41K128M16JT-125_AITK
- removed U67, U68, U69, U70: TLP785, Package_DIP:DIP-4_W7.62mm, symbol ebaz4205:TLP785
- removed U7: Micro_SD_Card_mount, symbol ebaz4205:Micro_SD_Card_mount
- removed U72: TPS51200AQDRCRQ1, TPS51200AQDRCRQ1, symbol ebaz4205:TPS51200AQDRCRQ1
- removed X3: DS1307Z+, SOIC127P600X175-8N, symbol ebaz4205:DS1307Z+
- removed X5: TXC-EBAZ, symbol ebaz4205:TXC-EBAZ
- removed X8: TXC-7C, Oscillator:Oscillator_SMD_TXC_7C-4Pin_5.0x3.2mm, symbol ebaz4205:TXC-7C
- removed Y2: RTC_XTAL, symbol ebaz4205:RTC_XTAL
- removed Y3: Crystal, symbol Device:Crystal
- added C9996: NC, symbol Device:C
- added C9997: 100NF, symbol Device:C
- added C9999: 33UF, symbol Device:C
- C2324, C2328, C2330, C2338, C2352, C2355: value C -> 3.9UF
- C2336, C2337, C2345, C2351, C2357, C2358: value C -> 51UF
- C2344: value C -> 33UF
- C2385, C325: value C -> 1NF
- C289, C290, C383, C385, C390, C392, C397, C399: value C -> 22UF
- C291, C292, C306, C309, C384, C389, C391, C396, C398, C403, C625, C626, C82: value C -> 10UF
- C293, C295, C320, C321, C387, C393, C394, C400, C401: value C -> 100NF
- C294, C386, C395, C402, C628, C845, C846, C856: value C -> NC
- D24: value D_ALT -> NC
- EC2, EC6: value CP -> 470UF/16V
- FB14: value L -> 1.2UH
- J4: value Conn_02x03_Odd_Even -> 2*3PIN-4.2MM
- L31, L32, L33, L37, L7: value L -> 4.7UH
- L36: value L -> 0.33UH
- LED4: value LED_ALT -> G
- R1333: value R_US -> 51K 5%
- R1336: value R_US -> 11.3K 1%
- R1373: value R_US -> 33R 1%
- R1413, R1415, R1418, R2599, R2800: value R_US -> 10K 1%
- R1414: value R_US -> 6.81K 1%
- R1417: value R_US -> 15K 1%
- R1420: value R_US -> 4.02K 1%
- R1421: value R_US -> 2K 1%
- R2468, R2487: value R_US -> NC
- R2471: value R_US -> 0R 5%
- R2558, R2559: value R_US -> 1M 5%
- R2603, R2604, R2605: value R_US -> 0R 1%
- R47: value R_US -> 150R 1%
- TP1: value TestPoint -> 3V3
- TP2: value TestPoint -> VDD_1V5
- TP3: value TestPoint -> 1V8
- TP4: value TestPoint -> 1V9
- U20, U21: value Q_NPN_BEC -> MMBT3904/1AM
- U23: value U23 -> NC
Connections:
- net GND: now also C9999.2
- net GNDADC_0: now also C9996.1
- net VCCP: now also C9999.1
- net VP1_0: now also C9996.2
- net NetL37_1: no longer names the net of J4.1 (Pin_1), J4.3 (Pin_3), J4.5 (Pin_5), L37.1
- net NetLED4_1: no longer names the net of LED4.2 (A), R47.2
- net NetR1373_2: no longer names the net of C625.1, R1373.2, U20.1 (B)
- net NetR1413_2: no longer names the net of C386.1, R1413.2, U26.5 (EN)
- net NetR2468_1: no longer names the net of R2468.1, R2487.2, U23.1
- net NetR2605_1: no longer names the net of R2605.1, U28.5 (EN)
- net NetR2800_2: no longer names the net of C402.1, C626.1, R2605.2, R2800.2, U21.3 (C)
- net NetU20_3: no longer names the net of C628.1, R2599.2, U20.3 (C), U21.1 (B)
- net NetU22_2: no longer names the net of C295.2, L7.2, U22.2 (SW)
- net NetU22_4: no longer names the net of R1333.2, R1336.1, U22.4 (FB)
- net NetU22_5: no longer names the net of C294.2, R2603.1, U22.5 (EN)
- net NetU22_6: no longer names the net of C295.1, U22.6 (S)
- net NetU26_2: no longer names the net of L31.1, U26.2 (SW)
- net NetU26_2: now also C9997.1
- net NetU26_4: no longer names the net of R1414.1, R1415.1, U26.4 (FB)
- net NetU26_6: no longer names the net of U26.6 (S)
- net NetU26_6: now also C9997.2
- net NetU27_2: no longer names the net of C393.2, L32.2, U27.2 (SW)
- net NetU27_4: no longer names the net of R1417.2, R1418.1, U27.4 (FB)
- net NetU27_5: no longer names the net of C395.2, R2604.1, U27.5 (EN)
- net NetU27_6: no longer names the net of C393.1, U27.6 (S)
- net NetU28_2: no longer names the net of C400.1, L33.1, U28.2 (SW)
- net NetU28_4: no longer names the net of R1420.1, R1421.1, U28.4 (FB)
- net NetU28_6: no longer names the net of C400.2, U28.6 (S)
Other:
- added sheet IO Sheet (IO.kicad_sch)
- added sheet Mem & Zynq Sheet (Mem_Zynq.kicad_sch)
- added sheet PHY & Sundries (Phy-Sun.kicad_sch)
- added sheet Zynq Power Sheet (Zynq_Pwr.kicad_sch)
- added sheet Zynq_IO Sheet (Zynq_IO.kicad_sch)
- note added: "+1V5 for DDR"
- note added: "+1V9 used for Zynq VCCBRAM, VCCINT and VCCPINT"
- note added: "High impeadance link between GNDs"
- note added: "Injection point for power from Data connectors"
- note added: "Main +3V3 rail."
- note added: "Main Power connector con only be used if D24 is fitted."
- note added: "Power Rails"
- note added: "Power on LED"
- note added: "R9999 was R120A R9998 was R2445B R9997 was R2473A R9996 was R2487A R9995 was R2641A C9999 was C2349A C9998 was C379A C9997 was C386A C9996 was C856A"
- note added: "This circuitry typically not fitted. Used to generate 1.25V for VREFP_0"
- note added: "VCC8 is used in opto isloator circuits"
- note added: "VCCA is 1V8 supply used for VCCAUX and VCCPAUX"
- note removed: "DDR"
- note removed: "DDR Termination"
- note removed: "Data Conns"
- note removed: "Ethernet PHY"
- note removed: "Flash"
- note removed: "Opto-Isolators"
- note removed: "Power"
- note removed: "RTC"
- note removed: "Reset Supervisor"
- note removed: "SD and Ancillary"
- note removed: "Switches"
- note removed: "Zynq"
- note removed: "Zynq IO"
- note removed: "Zynq Oscs"
- note removed: "Zynq Power"
- title: (none) -> EBAZ4205 Schematic rebuild.
